File: DIY/PS.sch (KiCad schematic (older format))
At the start: 6 parts, among them J1 PSX_PS2, J2 PSX_PS2, J3 DB25_Male, U1 AZ1117-5.0

Commit message: [DIY] Fixup N64 & PSX schematic
Parts:
- U1: value AZ1117-5.0 -> LT1117-5
Changed lines of the file:
@@
 P 4200 1800
 F 0 "U1" H 4200 2042 50  0000 C CNN
-F 1 "AZ1117-5.0" H 4200 1951 50  0000 C CNN
+F 1 "LT1117-5" H 4200 1951 50  0000 C CNN
 F 2 "" H 4200 2050 50  0001 C CIN
 F 3 "https://www.diodes.com/assets/Datasheets/AZ1117.pdf" H 4200 1800 50  0001 C CNN
