File: DevKit/BlueRetroCore.sch (KiCad schematic (older format))
At the start: 106 parts, among them J1 USB_C_Receptacle_USB2.0, J2 Conn_02x06, J3 Micro_SD_Card, J4 Conn_01x03, J5 DB25_Female, J6 Conn_02x13, J7 Conn_02x07, Q1 BSS138, Q2 BSS138, Q3 S8050, Q4 S8050, Q5 S8050, SW1 BOOT, SW2 EN, U1 ESP32-WROOM-32E, U10 TPD6F002DSVR, U11 TPD6F002DSVR, U12 TPD6F002DSVR, U13 TPD6F002DSVR, U2 FT2232HL, U3 STL6N3LLH6, U4 TCPP01-M12, U5 M93C46, U6 ECMF02-2AMX6, U7 TPD6F002DSVR, U8 AP7361C-33E, U9 AP7361C-33E, Y1 12MHz

Commit message: Simplify BR devkit
Parts:
- removed C17: 0.1u, BlueRetro:C_0402_1005Metric, symbol BlueRetro:C_Small
- removed D1, D8, D9: SS14, BlueRetro:D_SMA, symbol BlueRetro:D_SchottkyP
- removed D10: ESDA25P35-1U1M, BlueRetro:D_0603_1608Metric, symbol BlueRetro:D_Schottky
- removed D3: BAT54KFILM, BlueRetro:D_SOD-523, symbol BlueRetro:D_Schottky
- removed J3: Micro_SD_Card, BlueRetro:microSD_HC_Molex_104031-0811, symbol BlueRetro:Micro_SD_Card_Det
- removed J7: Conn_02x07, BlueRetro:PinHeader_2x07_P2.54mm_Vertical, symbol BlueRetro:Conn_02x07_Odd_Even
- removed R2: 0, BlueRetro:R_0603_1608Metric, symbol BlueRetro:R_0P
- removed R3: 10K, BlueRetro:R_0402_1005Metric, symbol BlueRetro:R_US
- removed R4: 2.7K, BlueRetro:R_0402_1005Metric, symbol BlueRetro:R_US
- removed U10, U11, U12, U13, U7: TPD6F002DSVR, BlueRetro:Texas_DVS_R-PWSON-N12, symbol BlueRetro:TPD6F003
- removed U3: STL6N3LLH6, BlueRetro:POWERFLAT-2X2, symbol BlueRetro:STL6N3LLH6
- removed U4: TCPP01-M12, BlueRetro:QFN-12-1EP_3x3mm_P0.5mm_EP1.65x1.65mm, symbol BlueRetro:TCPP01-M12
- removed U6: ECMF02-2AMX6, BlueRetro:ST_UQFN-6L_1.5x1.7mm_Pitch0.5mm, symbol BlueRetro:ECMF02-2AMX6
- added J3: SD_Card, Connector_Card:SD_Kyocera_145638009511859+, symbol BlueRetro:SD_Card
- added J7: Conn_01x07, Connector_PinHeader_2.54mm:PinHeader_1x07_P2.54mm_Vertical, symbol BlueRetro:Conn_01x07
- added R40, R41: 5.1K, BlueRetro:R_0402_1005Metric, symbol BlueRetro:R_US
Connections:
- net I34_C is gone; now on net I34: J5.10, J6.10 (Pin_10)
- net I35_C is gone; now on net I35: J5.23 (P23), J6.23 (Pin_23)
- net I36_C is gone; now on net I36: J5.21 (P21), J6.21 (Pin_21)
- net I39_C is gone; now on net I39: J5.22 (P22), J6.22 (Pin_22)
- net IO0_C is gone; now on net IO0: J5.20 (P20), J6.20 (Pin_20)
- net IO16_C is gone; now on net IO16: J5.19 (P19), J6.19 (Pin_19)
- net IO17_C is gone; now on net IO17: J5.18 (P18), J6.18 (Pin_18)
- net IO18_C is gone; now on net IO18: J5.4, J6.4 (Pin_4)
- net IO19_C is gone; now on net IO19: J5.16 (P16), J6.16 (Pin_16)
- net IO1_C is gone; now on net IO1: J5.2, J6.2 (Pin_2)
- net IO21_C is gone; now on net IO21: J5.3, J6.3 (Pin_3)
- net IO22_C is gone; now on net IO22: J5.14 (P14), J6.14 (Pin_14)
- net IO23_C is gone; now on net IO23: J5.1, J6.1 (Pin_1)
- net IO25_C is gone; now on net IO25: J5.12, J6.12 (Pin_12)
- net IO26_C is gone; now on net IO26: J5.25 (P25), J6.25 (Pin_25)
- net IO27_C is gone; now on net IO27: J5.13, J6.13 (Pin_13)
- net IO32_C is gone; now on net IO32: J5.11, J6.11 (Pin_11)
- net IO33_C is gone; now on net IO33: J5.24 (P24), J6.24 (Pin_24)
- net IO3_C is gone; now on net IO3: J5.15 (P15), J6.15 (Pin_15)
- net IO5_C is gone; now on net IO5: J5.17 (P17), J6.17 (Pin_17)
- net USB_N is gone; now on net USB_C_N: U2.7 (DM)
- net USB_P is gone; now on net USB_C_P: U2.8 (DP)
- net VIN_C is gone; now on net VIN: J5.7, J6.7 (Pin_7)
- net VOUT_C is gone; now on net +3V3: J5.6, J6.6 (Pin_6)
- net +3V3: now also U1.2 (3V3), J3.4 (VDD)
- net +3V3_USB: now also J7.1 (Pin_1)
- net GND: now also J3.12 (SHELL1), J3.13 (SHELL2), J3.3 (VSS), J3.6 (VSS), J7.7 (Pin_7), R40.1, R41.1
- net IO12: now also J3.9 (DAT2)
- net IO13: now also J3.1 (CD/DAT3)
- net IO14: now also J3.5 (CLK)
- net IO15: now also J3.2 (CMD)
- net IO2: now also J3.7 (DAT0)
- net IO4: now also J3.8 (DAT1)
- net TCK: now also J7.5 (Pin_5)
- net TDI: now also J7.6 (Pin_6)
- net TDO: now also J7.4 (Pin_4)
- net TMS: now also J7.3 (Pin_3)
- net VBUS: now also D2.1 (K), J1.A4 (VBUS), J1.A9 (VBUS), J1.B4 (VBUS), J1.B9 (VBUS)
- net nTRST: now also J7.2 (Pin_2)
- net at J1.A5 (CC1): now also R40.2
- net at J1.B5 (CC2): now also R41.2
- no-connect marks 40 -> 32
